Commit message: [synergy joint] modified the parent for the synergy joint

File: softhands_description/urdf/v2.0_simple/sh_v2_simple.xacro (robot description, xacro)
@@ -105,17 +105,4 @@
     <link name="${type}_hand_v2s_palm_base">
     </link>
-	<!-- synergy joint -->
-	<joint name="${type}_hand_v2s_synergy_joint" type="revolute">
-		<parent link="${type}_hand_v2s_palm_base"/>
-		<child link="${type}_hand_v2s_synergy_link"/>
-		<axis xyz="0 0 1"/>
-		<limit lower="${synergy_lb}" upper="${synergy_ub}" effort="${max_synergy_effort}" velocity="${max_synergy_velocity}"/>
-		<dynamics damping="${synergy_damping}" friction="${synergy_friction}"/>
-	</joint>
-	<link name="${type}_hand_v2s_synergy_link">
-		<inertial>
-			<xacro:insert_block name="negligible_inertia"/>
-		</inertial>
-	</link>
     # RIGHT HAND
     <xacro:if value="${type == 'right'}">
@@ -126,23 +113,23 @@
 	      <child link="${type}_hand_v2s_palm_link" />
       </joint>
-      <link name="${type}_hand_v2s_palm_link">
-	<inertial>
-	  <origin xyz="-0.004568758 -0.006808116 0.027653328"/>
-	  <mass value="0.266"/>
-	  <inertia ixx="0.001" ixy="0" ixz="0" iyy="0.001" iyz="0" izz="0.001"/>
-	</inertial>
-	<visual>
-	  <geometry>
-	    <mesh filename="package://softhands_description/meshes/softhands/v2.0/right/qbh_palm_ng.stl" scale="0.001 0.001 0.001"/>
-	  </geometry>
-	  <material name="qbmove/default"/>
-	</visual>
-	<collision>
-	  <geometry>
-	    <mesh filename="package://softhands_description/meshes/softhands/v2.0/right/qbh_palm_ng.stl" scale="0.001 0.001 0.001"/>
-	  </geometry>
-	</collision>
-      </link>
-      <gazebo reference="${type}_hand_v2s_palm_link">
+    <link name="${type}_hand_v2s_palm_link">
+		<inertial>
+		<origin xyz="-0.004568758 -0.006808116 0.027653328"/>
+		<mass value="0.266"/>
+		<inertia ixx="0.001" ixy="0" ixz="0" iyy="0.001" iyz="0" izz="0.001"/>
+		</inertial>
+		<visual>
+		<geometry>
+			<mesh filename="package://softhands_description/meshes/softhands/v2.0/right/qbh_palm_ng.stl" scale="0.001 0.001 0.001"/>
+		</geometry>
+		<material name="qbmove/default"/>
+		</visual>
+		<collision>
+		<geometry>
+			<mesh filename="package://softhands_description/meshes/softhands/v2.0/right/qbh_palm_ng.stl" scale="0.001 0.001 0.001"/>
+		</geometry>
+		</collision>
+    </link>
+    <gazebo reference="${type}_hand_v2s_palm_link">
       <material>Gazebo/Grey</material>
       <selfCollide>true</selfCollide>
@@ -318,4 +305,17 @@
       </xacro:finger_v2_simple>
     </xacro:if>
+	<!-- synergy joint -->
+	<joint name="${type}_hand_v2s_synergy_joint" type="revolute">
+		<parent link="${type}_hand_v2s_palm_link"/>
+		<child link="${type}_hand_v2s_synergy_link"/>
+		<axis xyz="0 0 1"/>
+		<limit lower="${synergy_lb}" upper="${synergy_ub}" effort="${max_synergy_effort}" velocity="${max_synergy_velocity}"/>
+		<dynamics damping="${synergy_damping}" friction="${synergy_friction}"/>
+	</joint>
+	<link name="${type}_hand_v2s_synergy_link">
+		<inertial>
+			<xacro:insert_block name="negligible_inertia"/>
+		</inertial>
+	</link>
 	  # Gazebo NEW custom synergy-plugin
 	  <gazebo>

Commit message: [grasp link] added grasp link

File: softhands_description/urdf/v2.0_simple/sh_v2_simple.xacro (robot description, xacro)
@@ -305,4 +305,18 @@
       </xacro:finger_v2_simple>
     </xacro:if>
+	<joint name="${type}_hand_v2s_grasp_joint" type="fixed">
+		<origin xyz="0 0 0.07" rpy="0 0 0"/>
+		<parent link="${type}_hand_v2s_palm_base"/>
+		<child link="${type}_hand_v2s_grasp_link"/>
+	</joint>
+	<link name="${type}_hand_v2s_grasp_link">
+		<inertial>
+			<xacro:insert_block name="negligible_inertia"/>
+		</inertial>
+	</link>
+	<gazebo reference="${type}_hand_v2s_grasp_link">
+		<material>Gazebo/Grey</material>
+		<selfCollide>true</selfCollide>
+	</gazebo>
 	<!-- synergy joint -->
 	<joint name="${type}_hand_v2s_synergy_joint" type="revolute">

Commit message: [multiplier] modified the multiplier to 1.2 for mimic joints

File: softhands_description/urdf/v2.0_simple/sh_v2_simple.xacro (robot description, xacro)
@@ -42,4 +42,8 @@
 	<!-- from pisa-iit soft hand description -->
 	<!-- pkg: pisa-iit-soft-hand/soft_hand_description/model/soft_hand.urdf.xacro -->
+	<!-- define material -->
+	<material name="qbmove/default">
+		<color rgba="0.5 0.5 0.5 1"/>
+	</material>
 	<!-- joint properties -->
 	<xacro:property name="abd_lb" value="-30" />
@@ -143,7 +147,7 @@
 	      damping="0.05"
 		  useMimicTag="${useMimicTag}"
-		  abd_R="1.0"
-		  inner_R="1.0"
-		  outer_R="1.0"
+		  abd_R="1.2"
+		  inner_R="1.2"
+		  outer_R="1.2"
 	      translation="${translation}"> <!-- added offset on orientation -->
       </xacro:thumb_v2_simple>
@@ -156,8 +160,8 @@
 	      damping="0.05"
 		  useMimicTag="${useMimicTag}"
-		  abd_R="1.0"
-		  inner_R="1.0"
-		  middle_R="1.0"
-		  outer_R="1.0"
+		  abd_R="1.2"
+		  inner_R="1.2"
+		  middle_R="1.2"
+		  outer_R="1.2"
 	      translation="${translation}">
       </xacro:finger_v2_simple>
@@ -170,8 +174,8 @@
 	      damping="0.05"
 		  useMimicTag="${useMimicTag}"
-		  abd_R="1.0"
-		  inner_R="1.0"
-		  middle_R="1.0"
-		  outer_R="1.0"
+		  abd_R="1.2"
+		  inner_R="1.2"
+		  middle_R="1.2"
+		  outer_R="1.2"
 	      translation="${translation}">
       </xacro:finger_v2_simple>
@@ -184,8 +188,8 @@
 	      damping="0.05"
 		  useMimicTag="${useMimicTag}"
-		  abd_R="1.0"
-		  inner_R="1.0"
-		  middle_R="1.0"
-		  outer_R="1.0"
+		  abd_R="1.2"
+		  inner_R="1.2"
+		  middle_R="1.2"
+		  outer_R="1.2"
 	      translation="${translation}">
       </xacro:finger_v2_simple>
@@ -198,8 +202,8 @@
 	      damping="0.05"
 		  useMimicTag="${useMimicTag}"
-		  abd_R="1.0"
-		  inner_R="1.0"
-		  middle_R="1.0"
-		  outer_R="1.0"
+		  abd_R="1.2"
+		  inner_R="1.2"
+		  middle_R="1.2"
+		  outer_R="1.2"
 	      translation="${translation}">
       </xacro:finger_v2_simple>
@@ -243,7 +247,7 @@
 	      damping="0.05"
 		  useMimicTag="${useMimicTag}"
-		  abd_R="1.0"
-		  inner_R="1.0"
-		  outer_R="1.0"
+		  abd_R="1.2"
+		  inner_R="1.2"
+		  outer_R="1.2"
 	      translation="${translation}">
       </xacro:thumb_v2_simple>
@@ -256,8 +260,8 @@
 	      damping="0.05"
 		  useMimicTag="${useMimicTag}"
-		  abd_R="1.0"
-		  inner_R="1.0"
-		  middle_R="1.0"
-		  outer_R="1.0"
+		  abd_R="1.2"
+		  inner_R="1.2"
+		  middle_R="1.2"
+		  outer_R="1.2"
 	      translation="${translation}">
       </xacro:finger_v2_simple>
@@ -270,8 +274,8 @@
 	      damping="0.05"
 		  useMimicTag="${useMimicTag}"
-		  abd_R="1.0"
-		  inner_R="1.0"
-		  middle_R="1.0"
-		  outer_R="1.0"
+		  abd_R="1.2"
+		  inner_R="1.2"
+		  middle_R="1.2"
+		  outer_R="1.2"
 	      translation="${translation}">
       </xacro:finger_v2_simple>
@@ -284,8 +288,8 @@
 	      damping="0.05"
 		  useMimicTag="${useMimicTag}"
-		  abd_R="1.0"
-		  inner_R="1.0"
-		  middle_R="1.0"
-		  outer_R="1.0"
+		  abd_R="1.2"
+		  inner_R="1.2"
+		  middle_R="1.2"
+		  outer_R="1.2"
 	      translation="${translation}">
       </xacro:finger_v2_simple>
@@ -298,8 +302,8 @@
 	      damping="0.05"
 		  useMimicTag="${useMimicTag}"
-		  abd_R="1.0"
-		  inner_R="1.0"
-		  middle_R="1.0"
-		  outer_R="1.0"
+		  abd_R="1.2"
+		  inner_R="1.2"
+		  middle_R="1.2"
+		  outer_R="1.2"
 	      translation="${translation}">
       </xacro:finger_v2_simple>
@@ -332,4 +336,30 @@
 		</inertial>
 	</link>
+	<gazebo reference="${type}_hand_v2s_synergy_link">
+		<material>Gazebo/Grey</material>
+		<collision name="${type}_hand_v2s_synergy_collision">
+			<surface>
+				<friction>
+					<torsional>
+						<coefficient>10.0</coefficient>
+						<use_patch_radius>true</use_patch_radius>
+						<patch_radius>0.05</patch_radius>
+					</torsional>
+				</friction>
+				<contact>
+					<poissons_ratio>0.5</poissons_ratio>
+					<elastic_modulus>1e8</elastic_modulus>
+				</contact>
+			</surface>
+		</collision>
+		<mu1>10</mu1>
+		<mu2>10</mu2>
+		<maxVel>1</maxVel>
+		<kp>1000000.0</kp>
+		<kd>100.0</kd>
+		<fdir1>0 0 1</fdir1>
+		<minDepth>0.0</minDepth>
+		<maxContacts>100</maxContacts>
+	</gazebo>
 	  # Gazebo NEW custom synergy-plugin
 	  <gazebo>
