Commit message: added fixed hand argument to v1 hand

File: softhands_description/urdf/softhands.xacro (robot description, xacro)
@@ -42,5 +42,5 @@
   <xacro:include filename="$(find softhands_description)/urdf/v2.0/sh_v2.xacro"/>
   <xacro:include filename="$(find softhands_description)/urdf/v2.0_simple/sh_v2_simple.xacro"/>
-  <xacro:macro name="softhands" params="type version parent position orientation operation_mode translation">
+  <xacro:macro name="softhands" params="type version parent position orientation operation_mode translation fixed_hands:='false'">
     # Softhand VERSION 1.0
     <xacro:if value="${version == 'v1.0'}">
@@ -58,5 +58,6 @@
         position ="${position}"
         orientation ="${orientation}"
-        operation_mode = "${operation_mode}">
+        operation_mode = "${operation_mode}"
+        fixed_hand = "${fixed_hands}">
       </xacro:sh_v1_simple>
     </xacro:if>

File: softhands_description/urdf/v1.0_simple/finger.xacro (robot description, xacro)
@@ -38,7 +38,13 @@
 -->
 <robot xmlns:xacro="http://www.ros.org/wiki/xacro">
-  <xacro:macro name="finger_v1_simple" params="type ns sign position orientation">
+  <xacro:macro name="finger_v1_simple" params="type ns sign position orientation fixed:='false'">
+  <xacro:if value="${fixed == False}">
+    <xacro:property name="joint_type" value="revolute"/>
+  </xacro:if>
+  <xacro:if value="${fixed == True}">
+    <xacro:property name="joint_type" value="fixed"/>
+  </xacro:if>
     <!-- KNUCKLE -->
-    <joint name="${ns}_${type}_knuckle_joint" type="revolute">
+    <joint name="${ns}_${type}_knuckle_joint" type="${joint_type}">
       <origin xyz="${position}" rpy="${orientation}"/>
       <parent link="${ns}_palm_link"/>
@@ -66,5 +72,5 @@
     </link>
     <!-- PROXIMAL PHALANGE -->
-    <joint name="${ns}_${type}_proximal_joint" type="revolute">
+    <joint name="${ns}_${type}_proximal_joint" type="${joint_type}">
       <origin xyz="0.020 0 0" rpy="0 0 0" />
       <parent link="${ns}_${type}_knuckle_link"/>
@@ -91,5 +97,5 @@
     </link>
     <!-- MIDDLE PHALANGE -->
-    <joint name="${ns}_${type}_middle_joint" type="revolute">
+    <joint name="${ns}_${type}_middle_joint" type="${joint_type}">
       <origin xyz="0.020 0 0" rpy="0 0 0" />
       <parent link="${ns}_${type}_proximal_link"/>
@@ -117,5 +123,5 @@
     </link>
     <!-- DISTAL PHALANGE -->
-    <joint name="${ns}_${type}_distal_joint" type="revolute">
+    <joint name="${ns}_${type}_distal_joint" type="${joint_type}">
       <origin xyz="0.020 0 0" rpy="0 0 0" />
       <parent link="${ns}_${type}_middle_link"/>

File: softhands_description/urdf/v1.0_simple/sh_v1_simple.xacro (robot description, xacro)
@@ -40,5 +40,5 @@
 	<xacro:include filename="$(find softhands_description)/urdf/v1.0_simple/finger.xacro" />
 	<xacro:include filename="$(find softhands_description)/urdf/v1.0_simple/thumb.xacro" />
-	<xacro:macro name="sh_v1_simple" params="type parent position orientation operation_mode">
+	<xacro:macro name="sh_v1_simple" params="type parent position orientation operation_mode fixed_hand:='false'">
 		# Softhand Base
 		<joint name="${type}_hand_base_joint" type="fixed">
@@ -86,13 +86,13 @@
 			</link>
 			# Thumb finger
-			<xacro:thumb_v1_simple type="thumb" ns="${type}_hand_v1s" sign="1" position="0.00566972 0.0296160 0.0553140" orientation="0.0 -0.38397275793662144 1.5707963267948966"></xacro:thumb_v1_simple>
+			<xacro:thumb_v1_simple type="thumb" ns="${type}_hand_v1s" sign="1" position="0.00566972 0.0296160 0.0553140" orientation="0.0 -0.38397275793662144 1.5707963267948966" fixed="${fixed_hand}"></xacro:thumb_v1_simple>
 			# Index finger
-			<xacro:finger_v1_simple type="index" ns="${type}_hand_v1s" sign="1" position="-0.0033 0.0195 0.0936994" orientation="1.5707963267948966 -1.4835299330931884 1.5707963267948966"></xacro:finger_v1_simple>
+			<xacro:finger_v1_simple type="index" ns="${type}_hand_v1s" sign="1" position="-0.0033 0.0195 0.0936994" orientation="1.5707963267948966 -1.4835299330931884 1.5707963267948966" fixed="${fixed_hand}"></xacro:finger_v1_simple>
 			# Middle finger
-			<xacro:finger_v1_simple type="middle" ns="${type}_hand_v1s" sign="1" position="-0.003300000 0.0 0.100699" orientation="3.141592 -1.5707963267948966 0.0"></xacro:finger_v1_simple>
+			<xacro:finger_v1_simple type="middle" ns="${type}_hand_v1s" sign="1" position="-0.003300000 0.0 0.100699" orientation="3.141592 -1.5707963267948966 0.0" fixed="${fixed_hand}"></xacro:finger_v1_simple>
 			# Ring finger
-			<xacro:finger_v1_simple type="ring" ns="${type}_hand_v1s" sign="1" position="-0.0033 -0.0195 0.0936994" orientation="-1.5707963267948966 -1.5184364298870514 -1.5707963267948966"></xacro:finger_v1_simple>
+			<xacro:finger_v1_simple type="ring" ns="${type}_hand_v1s" sign="1" position="-0.0033 -0.0195 0.0936994" orientation="-1.5707963267948966 -1.5184364298870514 -1.5707963267948966" fixed="${fixed_hand}"></xacro:finger_v1_simple>
 			# Little finger
-			<xacro:finger_v1_simple type="little" ns="${type}_hand_v1s" sign="1" position="-0.0033 -0.039 0.0836994" orientation="-1.5707963267948966 -1.4835299330931884 -1.5707963267948966"></xacro:finger_v1_simple>
+			<xacro:finger_v1_simple type="little" ns="${type}_hand_v1s" sign="1" position="-0.0033 -0.039 0.0836994" orientation="-1.5707963267948966 -1.4835299330931884 -1.5707963267948966" fixed="${fixed_hand}"></xacro:finger_v1_simple>
 		</xacro:if>
 		# LEFT HAND
@@ -134,13 +134,13 @@
 			</link>
 			# Thumb finger
-			<xacro:thumb_v1_simple type="thumb" ns="${type}_hand_v1s" sign="-1" position="0.005669722 -0.029616 0.055314" orientation="0.0 -0.38397275793662144 -1.5707963267948966"></xacro:thumb_v1_simple>
+			<xacro:thumb_v1_simple type="thumb" ns="${type}_hand_v1s" sign="-1" position="0.005669722 -0.029616 0.055314" orientation="0.0 -0.38397275793662144 -1.5707963267948966" fixed="${fixed_hand}"></xacro:thumb_v1_simple>
 			# Index finger
-			<xacro:finger_v1_simple type="index" ns="${type}_hand_v1s" sign="-1" position="-0.0033 -0.0195 0.0936994" orientation="-1.5707963267948966 -1.4835299330931884 -1.5707963267948966"></xacro:finger_v1_simple>
+			<xacro:finger_v1_simple type="index" ns="${type}_hand_v1s" sign="-1" position="-0.0033 -0.0195 0.0936994" orientation="-1.5707963267948966 -1.4835299330931884 -1.5707963267948966" fixed="${fixed_hand}"></xacro:finger_v1_simple>
 			# Middle finger
-			<xacro:finger_v1_simple type="middle" ns="${type}_hand_v1s" sign="-1" position="-0.0033 0.0 0.100699" orientation="3.1415 -1.5707963267948966 0.0"></xacro:finger_v1_simple>
+			<xacro:finger_v1_simple type="middle" ns="${type}_hand_v1s" sign="-1" position="-0.0033 0.0 0.100699" orientation="3.1415 -1.5707963267948966 0.0" fixed="${fixed_hand}"></xacro:finger_v1_simple>
 			# Ring finger
-			<xacro:finger_v1_simple type="ring" ns="${type}_hand_v1s" sign="-1" position="-0.0033 0.0195 0.0936994" orientation="1.5707963267948966 -1.5184364298870514 1.5707963267948966"></xacro:finger_v1_simple>
+			<xacro:finger_v1_simple type="ring" ns="${type}_hand_v1s" sign="-1" position="-0.0033 0.0195 0.0936994" orientation="1.5707963267948966 -1.5184364298870514 1.5707963267948966" fixed="${fixed_hand}"></xacro:finger_v1_simple>
 			# Little finger
-			<xacro:finger_v1_simple type="little" ns="${type}_hand_v1s" sign="-1" position="-0.0033 0.039 0.0836994" orientation="1.5707963267948966 -1.4835299330931884 1.5707963267948966"></xacro:finger_v1_simple>
+			<xacro:finger_v1_simple type="little" ns="${type}_hand_v1s" sign="-1" position="-0.0033 0.039 0.0836994" orientation="1.5707963267948966 -1.4835299330931884 1.5707963267948966" fixed="${fixed_hand}"></xacro:finger_v1_simple>
 		</xacro:if>
 		# Gazebo NEW custom synergy-plugin

File: softhands_description/urdf/v1.0_simple/thumb.xacro (robot description, xacro)
@@ -38,7 +38,13 @@
 -->
 <robot xmlns:xacro="http://www.ros.org/wiki/xacro">
-  <xacro:macro name="thumb_v1_simple" params="type ns sign position orientation">
+  <xacro:macro name="thumb_v1_simple" params="type ns sign position orientation fixed:='false'">
+  <xacro:if value="${fixed == False}">
+    <xacro:property name="joint_type" value="continuous"/>
+  </xacro:if>
+  <xacro:if value="${fixed == True}">
+    <xacro:property name="joint_type" value="fixed"/>
+  </xacro:if>
     <!-- KNUCKLE -->
-    <joint name="${ns}_${type}_knuckle_joint" type="continuous">
+    <joint name="${ns}_${type}_knuckle_joint" type="${joint_type}">
       <origin xyz="${position}" rpy="${orientation}"/>
       <parent link="${ns}_palm_link"/>
@@ -79,5 +85,5 @@
     </link>
     <!-- PROXIMAL PHALANGE -->
-    <joint name="${ns}_${type}_proximal_joint" type="continuous">
+    <joint name="${ns}_${type}_proximal_joint" type="${joint_type}">
       <origin xyz="0.033500000 ${sign*-0.003300000} 0.0" rpy="${sign*0.426627741408745} 0 0.0" />
       <parent link="${ns}_${type}_knuckle_link"/>
@@ -104,5 +110,5 @@
     </link>
     <!-- DISTAL PHALANGE -->
-    <joint name="${ns}_${type}_distal_joint" type="continuous">
+    <joint name="${ns}_${type}_distal_joint" type="${joint_type}">
       <origin xyz="0.020 0 0.0" rpy="0 0 0" />
       <parent link="${ns}_${type}_proximal_link"/>

Commit message: [synergy_joint] added mimic tags for synergy joint

File: softhands_description/urdf/softhands.xacro (robot description, xacro)
@@ -42,5 +42,5 @@
   <xacro:include filename="$(find softhands_description)/urdf/v2.0/sh_v2.xacro"/>
   <xacro:include filename="$(find softhands_description)/urdf/v2.0_simple/sh_v2_simple.xacro"/>
-  <xacro:macro name="softhands" params="type version parent position orientation operation_mode translation fixed_hands:='false'">
+  <xacro:macro name="softhands" params="type version parent position orientation operation_mode translation useMimicTag fixed_hands:='false'">
     # Softhand VERSION 1.0
     <xacro:if value="${version == 'v1.0'}">
@@ -75,4 +75,5 @@
       <xacro:sh_v2_simple type="${type}"
 	      parent = "${parent}"
+        useMimicTag="${useMimicTag}"
 	      position ="${position}"
 	      orientation ="${orientation}"

File: softhands_description/urdf/v2.0_simple/finger.xacro (robot description, xacro)
@@ -38,5 +38,5 @@
 -->
 <robot xmlns:xacro="http://www.ros.org/wiki/xacro">
-  <xacro:macro name="finger_v2_simple" params="type ns sign position orientation translation damping">
+  <xacro:macro name="finger_v2_simple" params="type ns sign position orientation translation damping useMimicTag abd_R inner_R middle_R outer_R">
     <!-- KNUCKLE -->
     <joint name="${ns}_${type}_knuckle_joint" type="revolute">
@@ -47,4 +47,7 @@
       <dynamics damping="${damping}" friction="0.0" />
       <axis xyz="0 0 1" />
+	  <xacro:if value="${useMimicTag}">
+        <mimic joint="${ns}_synergy_joint" multiplier="${abd_R}" />
+      </xacro:if>
     </joint>
     <link name="${ns}_${type}_knuckle_link">
@@ -179,4 +182,7 @@
       <dynamics damping="${damping}" friction="0.0" />
       <axis xyz="0 0 1" />
+	  <xacro:if value="${useMimicTag}">
+        <mimic joint="${ns}_synergy_joint" multiplier="${inner_R}" />
+      </xacro:if>
     </joint>
      <link name="${ns}_${type}_proximal_link">
@@ -221,4 +227,7 @@
       <dynamics damping="${damping}" friction="0.0" />
       <axis xyz="0 0 1" />
+	  <xacro:if value="${useMimicTag}">
+        <mimic joint="${ns}_synergy_joint" multiplier="${middle_R}" />
+      </xacro:if>
     </joint>
     <link name="${ns}_${type}_middle_link">
@@ -263,4 +272,7 @@
       <dynamics damping="${damping}" friction="0.0" />
       <axis xyz="0 0 1" />
+	  <xacro:if value="${useMimicTag}">
+        <mimic joint="${ns}_synergy_joint" multiplier="${outer_R}" />
+      </xacro:if>
     </joint>
     <link name="${ns}_${type}_distal_link">

File: softhands_description/urdf/v2.0_simple/sh_v2_simple.xacro (robot description, xacro)
@@ -40,5 +40,61 @@
   <xacro:include filename="$(find softhands_description)/urdf/v2.0_simple/finger.xacro"/>
   <xacro:include filename="$(find softhands_description)/urdf/v2.0_simple/thumb.xacro"/>
-  <xacro:macro name="sh_v2_simple" params="type parent position orientation operation_mode translation">
+	<!-- from pisa-iit soft hand description -->
+	<!-- pkg: pisa-iit-soft-hand/soft_hand_description/model/soft_hand.urdf.xacro -->
+	<!-- joint properties -->
+	<xacro:property name="abd_lb" value="-30" />
+	<xacro:property name="abd_ub" value="30" />
+	<xacro:property name="thumb_abd_lb" value="0" />
+	<xacro:property name="thumb_abd_ub" value="90" />
+	<xacro:property name="inner_lb" value="0" />
+	<xacro:property name="inner_ub" value="45" />
+	<xacro:property name="middle_lb" value="0" />
+	<xacro:property name="middle_ub" value="45" />
+	<xacro:property name="outer_lb" value="0" />
+	<xacro:property name="outer_ub" value="45" />
+	<xacro:property name="velocity" value="100" />
+	<xacro:property name="effort" value="100" />
+	<xacro:property name="damping" value="0.0" />
+	<xacro:property name="friction" value="0.0" />
+	<!-- synergy vector -->
+	<xacro:property name="syn_amp" value="1" />
+	<xacro:property name="thumb_abd_R" value="${1.3*syn_amp}" />
+	<xacro:property name="thumb_inner_R" value="${1.3*syn_amp}" />
+	<xacro:property name="thumb_outer_R" value="${1.0*syn_amp}" />
+	<xacro:property name="index_abd_R" value="-${0.2*syn_amp}" />
+	<xacro:property name="index_inner_R" value="${1.0*syn_amp}" />
+	<xacro:property name="index_middle_R" value="${1.0*syn_amp}" />
+	<xacro:property name="index_outer_R" value="${1.0*syn_amp}" />
+	<xacro:property name="middle_abd_R" value="${0.0*syn_amp}" />
+	<xacro:property name="middle_inner_R" value="${1.0*syn_amp}" />
+	<xacro:property name="middle_middle_R" value="${1.0*syn_amp}" />
+	<xacro:property name="middle_outer_R" value="${1.0*syn_amp}" />
+	<xacro:property name="ring_abd_R" value="${0.2*syn_amp}" />
+	<xacro:property name="ring_inner_R" value="${1.0*syn_amp}" />
+	<xacro:property name="ring_middle_R" value="${1.0*syn_amp}" />
+	<xacro:property name="ring_outer_R" value="${1.0*syn_amp}" />
+	<xacro:property name="little_abd_R" value="${0.4*syn_amp}" />
+	<xacro:property name="little_inner_R" value="${1.0*syn_amp}" />
+	<xacro:property name="little_middle_R" value="${1.0*syn_amp}" />
+	<xacro:property name="little_outer_R" value="${1.0*syn_amp}" />
+  	<!-- conversions -->
+    <xacro:property name="mm_to_m" value="0.001"/>
+    <xacro:property name="mm2_to_m2" value="0.001"/>
+    <xacro:property name="gr_to_Kg" value="0.01"/>
+    <!-- not so negligible, otherwise simulation fails -->
+    <xacro:property name="negligible_mass" value="${10*gr_to_Kg}"/>
+    <xacro:property name="negligible_inertia">
+        <origin xyz="0 0 0"/>
+        <mass value="${negligible_mass}"/>
+        <inertia ixx="${negligible_mass * 10 * mm2_to_m2}" ixy="0.0" ixz="0.0" iyy="${negligible_mass * 10 * mm2_to_m2}" iyz="0.0" izz="${negligible_mass * 10 * mm2_to_m2}"/>
+    </xacro:property>
+  	<!-- synergy joint properties -->
+	<xacro:property name="synergy_lb" value="0.0" />
+	<xacro:property name="synergy_ub" value="1.0"/>
+	<xacro:property name="max_synergy_velocity" value="100000" />
+	<xacro:property name="max_synergy_effort" value="100" />
+	<xacro:property name="synergy_damping" value="0.0" />
+	<xacro:property name="synergy_friction" value="0.0" />
+  <xacro:macro name="sh_v2_simple" params="type parent position orientation operation_mode translation useMimicTag">
     # Softhand Base
     <joint name="${type}_hand_v2s_base_joint" type="fixed">
@@ -49,4 +105,17 @@
     <link name="${type}_hand_v2s_palm_base">
     </link>
+	<!-- synergy joint -->
+	<joint name="${type}_hand_v2s_synergy_joint" type="revolute">
+		<parent link="${type}_hand_v2s_palm_base"/>
+		<child link="${type}_hand_v2s_synergy_link"/>
+		<axis xyz="0 0 1"/>
+		<limit lower="${synergy_lb}" upper="${synergy_ub}" effort="${max_synergy_effort}" velocity="${max_synergy_velocity}"/>
+		<dynamics damping="${synergy_damping}" friction="${synergy_friction}"/>
+	</joint>
+	<link name="${type}_hand_v2s_synergy_link">
+		<inertial>
+			<xacro:insert_block name="negligible_inertia"/>
+		</inertial>
+	</link>
     # RIGHT HAND
     <xacro:if value="${type == 'right'}">
@@ -86,4 +155,8 @@
 	      orientation="-1.5707963 -0.7 -1.0471972"
 	      damping="0.05"
+		  useMimicTag="${useMimicTag}"
+		  abd_R="${thumb_abd_R *(thumb_abd_ub - thumb_abd_lb)*pi/180}"
+		  inner_R="${thumb_inner_R *(inner_ub - inner_lb)*pi/180}"
+		  outer_R="${thumb_outer_R *(outer_ub - outer_lb)*pi/180}"
 	      translation="${translation}"> <!-- added offset on orientation -->
       </xacro:thumb_v2_simple>
@@ -95,4 +168,9 @@
 	      orientation="0 0 -0.1745327"
 	      damping="0.05"
+		  useMimicTag="${useMimicTag}"
+		  abd_R="${index_abd_R}"
+		  inner_R="${index_inner_R *(inner_ub - inner_lb)*pi/180}"
+		  middle_R="${index_middle_R *(middle_ub - middle_lb)*pi/180}"
+		  outer_R="${index_outer_R *(outer_ub - outer_lb)*pi/180}"
 	      translation="${translation}">
       </xacro:finger_v2_simple>
@@ -104,4 +182,9 @@
 	      orientation="0.0 0.0 0.0"
 	      damping="0.05"
+		  useMimicTag="${useMimicTag}"
+		  abd_R="${middle_abd_R}"
+		  inner_R="${middle_inner_R *(inner_ub - inner_lb)*pi/180}"
+		  middle_R="${middle_middle_R *(middle_ub - middle_lb)*pi/180}"
+		  outer_R="${middle_outer_R *(outer_ub - outer_lb)*pi/180}"
 	      translation="${translation}">
       </xacro:finger_v2_simple>
@@ -113,4 +196,9 @@
 	      orientation="0 0 0.0872664"
 	      damping="0.05"
+		  useMimicTag="${useMimicTag}"
+		  abd_R="${ring_abd_R}"
+		  inner_R="${ring_inner_R *(inner_ub - inner_lb)*pi/180}"
+		  middle_R="${ring_middle_R *(middle_ub - middle_lb)*pi/180}"
+		  outer_R="${ring_outer_R *(outer_ub - outer_lb)*pi/180}"
 	      translation="${translation}">
       </xacro:finger_v2_simple>
@@ -122,4 +210,9 @@
 	      orientation="0 0 0.2617993"
 	      damping="0.05"
+		  useMimicTag="${useMimicTag}"
+		  abd_R="${little_abd_R}"
+		  inner_R="${little_inner_R *(inner_ub - inner_lb)*pi/180}"
+		  middle_R="${little_middle_R *(middle_ub - middle_lb)*pi/180}"
+		  outer_R="${little_outer_R *(outer_ub - outer_lb)*pi/180}"
 	      translation="${translation}">
       </xacro:finger_v2_simple>
@@ -162,4 +255,8 @@
 	      orientation="1.5707963 0 1.0471971"
 	      damping="0.05"
+		  useMimicTag="${useMimicTag}"
+		  abd_R="${thumb_abd_R *(thumb_abd_ub - thumb_abd_lb)*pi/180}"
+		  inner_R="${thumb_inner_R *(inner_ub - inner_lb)*pi/180}"
+		  outer_R="${thumb_outer_R *(outer_ub - outer_lb)*pi/180}"
 	      translation="${translation}">
       </xacro:thumb_v2_simple>
@@ -171,4 +268,9 @@
 	      orientation="0 0 0.1745327"
 	      damping="0.05"
+		  useMimicTag="${useMimicTag}"
+		  abd_R="${index_abd_R}"
+		  inner_R="${index_inner_R *(inner_ub - inner_lb)*pi/180}"
+		  middle_R="${index_middle_R *(middle_ub - middle_lb)*pi/180}"
+		  outer_R="${index_outer_R *(outer_ub - outer_lb)*pi/180}"
 	      translation="${translation}">
       </xacro:finger_v2_simple>
@@ -180,4 +282,9 @@
 	      orientation="0.0 0.0 0.0"
 	      damping="0.05"
+		  useMimicTag="${useMimicTag}"
+		  abd_R="${middle_abd_R}"
+		  inner_R="${middle_inner_R *(inner_ub - inner_lb)*pi/180}"
+		  middle_R="${middle_middle_R *(middle_ub - middle_lb)*pi/180}"
+		  outer_R="${middle_outer_R *(outer_ub - outer_lb)*pi/180}"
 	      translation="${translation}">
       </xacro:finger_v2_simple>
@@ -189,4 +296,9 @@
 	      orientation="0 0 -0.0872667 "
 	      damping="0.05"
+		  useMimicTag="${useMimicTag}"
+		  abd_R="${ring_abd_R}"
+		  inner_R="${ring_inner_R *(inner_ub - inner_lb)*pi/180}"
+		  middle_R="${ring_middle_R *(middle_ub - middle_lb)*pi/180}"
+		  outer_R="${ring_outer_R *(outer_ub - outer_lb)*pi/180}"
 	      translation="${translation}">
       </xacro:finger_v2_simple>
@@ -198,4 +310,9 @@
 	      orientation="0 0 -0.2617993"
 	      damping="0.05"
+		  useMimicTag="${useMimicTag}"
+		  abd_R="${little_abd_R}"
+		  inner_R="${little_inner_R *(inner_ub - inner_lb)*pi/180}"
+		  middle_R="${little_middle_R *(middle_ub - middle_lb)*pi/180}"
+		  outer_R="${little_outer_R *(outer_ub - outer_lb)*pi/180}"
 	      translation="${translation}">
       </xacro:finger_v2_simple>

File: softhands_description/urdf/v2.0_simple/thumb.xacro (robot description, xacro)
@@ -38,5 +38,5 @@
 -->
 <robot xmlns:xacro="http://www.ros.org/wiki/xacro">
-  <xacro:macro name="thumb_v2_simple" params="type ns sign position orientation translation damping">
+  <xacro:macro name="thumb_v2_simple" params="type ns sign position orientation translation damping useMimicTag abd_R inner_R outer_R">
     <!-- KNUCKLE -->
     <joint name="${ns}_${type}_knuckle_joint" type="revolute">
@@ -47,4 +47,7 @@
       <limit effort="30" velocity="1.0" lower="0" upper="1.57" />
       <dynamics damping="${damping}" friction="0.0" />
+      <xacro:if value="${useMimicTag}">
+        <mimic joint="${ns}_synergy_joint" multiplier="${abd_R}" />
+      </xacro:if>
     </joint>
     <link name="${ns}_${type}_knuckle_link">
@@ -99,4 +102,7 @@
       <limit effort="30" velocity="1.0" lower="-0.785398" upper="1.57" />
       <dynamics damping="${damping}" friction="0.0" />
+      <xacro:if value="${useMimicTag}">
+        <mimic joint="${ns}_synergy_joint" multiplier="${inner_R}" />
+      </xacro:if>
     </joint>
     <link name="${ns}_${type}_proximal_link">
@@ -141,4 +147,7 @@
       <axis xyz="0 0 1" />
       <dynamics damping="${damping}" friction="0.0" />
+      <xacro:if value="${useMimicTag}">
+        <mimic joint="${ns}_synergy_joint" multiplier="${outer_R}" />
+      </xacro:if>
     </joint>
     <link name="${ns}_${type}_distal_link">
