Commit message: [gazebo] added gazebo plugins for mimic joints

File: softhands_description/urdf/softhands.xacro (robot description, xacro)
@@ -42,5 +42,5 @@
   <xacro:include filename="$(find softhands_description)/urdf/v2.0/sh_v2.xacro"/>
   <xacro:include filename="$(find softhands_description)/urdf/v2.0_simple/sh_v2_simple.xacro"/>
-  <xacro:macro name="softhands" params="type version parent position orientation operation_mode translation useMimicTag fixed_hands:='false'">
+  <xacro:macro name="softhands" params="type version parent position orientation operation_mode translation useMimicTag:='false' fixed_hands:='false'">
     # Softhand VERSION 1.0
     <xacro:if value="${version == 'v1.0'}">

File: softhands_description/urdf/v2.0_simple/finger.xacro (robot description, xacro)
@@ -39,4 +39,22 @@
 <robot xmlns:xacro="http://www.ros.org/wiki/xacro">
   <xacro:macro name="finger_v2_simple" params="type ns sign position orientation translation damping useMimicTag abd_R inner_R middle_R outer_R">
+	<xacro:macro name="mimic_joint_plugin_gazebo" params="name_prefix parent_joint mimic_joint has_pid:=false multiplier:=1.0 offset:=0 sensitiveness:=0.0 max_effort:=1.0">
+      <gazebo>
+        <plugin name="${name_prefix}mimic_joint_plugin" filename="libroboticsgroup_upatras_gazebo_mimic_joint_plugin.so">
+          <joint>${parent_joint}</joint>
+          <mimicJoint>${mimic_joint}</mimicJoint>
+          <xacro:if value="${has_pid}">                     <!-- if set to true, PID parameters from "/gazebo_ros_control/pid_gains/${mimic_joint}" are loaded -->
+            <hasPID />
+          </xacro:if>
+          <multiplier>${multiplier}</multiplier>
+          <offset>${offset}</offset>
+          <sensitiveness>${sensitiveness}</sensitiveness>   <!-- if absolute difference between setpoint and process value is below this threshold, do nothing; 0.0 = disable [rad] -->
+          <maxEffort>${max_effort}</maxEffort>              <!-- only taken into account if has_pid:=true [Nm] -->
+          <xacro:unless value="${ns == ''}">
+            <robotNamespace>${ns}</robotNamespace>
+          </xacro:unless>
+        </plugin>
+      </gazebo>
+    </xacro:macro>
     <!-- KNUCKLE -->
     <joint name="${ns}_${type}_knuckle_joint" type="revolute">
@@ -51,4 +69,9 @@
       </xacro:if>
     </joint>
+	<xacro:if value="${useMimicTag}">
+	  <xacro:mimic_joint_plugin_gazebo name_prefix="${ns}_${type}_knuckle_joint"
+	  	parent_joint="${ns}_synergy_joint" mimic_joint="${ns}_${type}_knuckle_joint"
+		has_pid="true" multiplier="${abd_R}" />
+	</xacro:if>
     <link name="${ns}_${type}_knuckle_link">
       <inertial>
@@ -186,4 +209,9 @@
       </xacro:if>
     </joint>
+	<xacro:if value="${useMimicTag}">
+	  <xacro:mimic_joint_plugin_gazebo name_prefix="${ns}_${type}_proximal_joint"
+	  	parent_joint="${ns}_synergy_joint" mimic_joint="${ns}_${type}_proximal_joint"
+		has_pid="true" multiplier="${abd_R}" />
+	</xacro:if>
      <link name="${ns}_${type}_proximal_link">
       <inertial>
@@ -231,4 +259,9 @@
       </xacro:if>
     </joint>
+	<xacro:if value="${useMimicTag}">
+	  <xacro:mimic_joint_plugin_gazebo name_prefix="${ns}_${type}_middle_joint"
+	  	parent_joint="${ns}_synergy_joint" mimic_joint="${ns}_${type}_middle_joint"
+		has_pid="true" multiplier="${abd_R}" />
+	</xacro:if>
     <link name="${ns}_${type}_middle_link">
       <inertial>
@@ -276,4 +309,9 @@
       </xacro:if>
     </joint>
+	<xacro:if value="${useMimicTag}">
+	  <xacro:mimic_joint_plugin_gazebo name_prefix="${ns}_${type}_distal_joint"
+	  	parent_joint="${ns}_synergy_joint" mimic_joint="${ns}_${type}_distal_joint"
+		has_pid="true" multiplier="${abd_R}" />
+	</xacro:if>
     <link name="${ns}_${type}_distal_link">
       <inertial>

File: softhands_description/urdf/v2.0_simple/thumb.xacro (robot description, xacro)
@@ -39,4 +39,22 @@
 <robot xmlns:xacro="http://www.ros.org/wiki/xacro">
   <xacro:macro name="thumb_v2_simple" params="type ns sign position orientation translation damping useMimicTag abd_R inner_R outer_R">
+    <xacro:macro name="mimic_joint_plugin_gazebo" params="name_prefix parent_joint mimic_joint has_pid:=false multiplier:=1.0 offset:=0 sensitiveness:=0.0 max_effort:=1.0">
+      <gazebo>
+        <plugin name="${name_prefix}mimic_joint_plugin" filename="libroboticsgroup_upatras_gazebo_mimic_joint_plugin.so">
+          <joint>${parent_joint}</joint>
+          <mimicJoint>${mimic_joint}</mimicJoint>
+          <xacro:if value="${has_pid}">                     <!-- if set to true, PID parameters from "/gazebo_ros_control/pid_gains/${mimic_joint}" are loaded -->
+            <hasPID />
+          </xacro:if>
+          <multiplier>${multiplier}</multiplier>
+          <offset>${offset}</offset>
+          <sensitiveness>${sensitiveness}</sensitiveness>   <!-- if absolute difference between setpoint and process value is below this threshold, do nothing; 0.0 = disable [rad] -->
+          <maxEffort>${max_effort}</maxEffort>              <!-- only taken into account if has_pid:=true [Nm] -->
+          <xacro:unless value="${ns == ''}">
+            <robotNamespace>${ns}</robotNamespace>
+          </xacro:unless>
+        </plugin>
+      </gazebo>
+    </xacro:macro>
     <!-- KNUCKLE -->
     <joint name="${ns}_${type}_knuckle_joint" type="revolute">
@@ -51,4 +69,7 @@
       </xacro:if>
     </joint>
+    <xacro:mimic_joint_plugin_gazebo name_prefix="${ns}_${type}_knuckle_joint"
+      parent_joint="${ns}_synergy_joint" mimic_joint="${ns}_${type}_knuckle_joint"
+      has_pid="true" multiplier="${abd_R}" />
     <link name="${ns}_${type}_knuckle_link">
       <inertial>
@@ -106,4 +127,7 @@
       </xacro:if>
     </joint>
+    <xacro:mimic_joint_plugin_gazebo name_prefix="${ns}_${type}_proximal_joint"
+      parent_joint="${ns}_synergy_joint" mimic_joint="${ns}_${type}_proximal_joint"
+      has_pid="true" multiplier="${inner_R}" />
     <link name="${ns}_${type}_proximal_link">
       <inertial>
@@ -151,4 +175,7 @@
       </xacro:if>
     </joint>
+    <xacro:mimic_joint_plugin_gazebo name_prefix="${ns}_${type}_distal_joint"
+      parent_joint="${ns}_synergy_joint" mimic_joint="${ns}_${type}_distal_joint"
+      has_pid="true" multiplier="${outer_R}" />
     <link name="${ns}_${type}_distal_link">
       <inertial>

Commit message: added flag to disable collision meshes for dawnik

File: softhands_description/urdf/softhands.xacro (robot description, xacro)
@@ -42,5 +42,5 @@
   <xacro:include filename="$(find softhands_description)/urdf/v2.0/sh_v2.xacro"/>
   <xacro:include filename="$(find softhands_description)/urdf/v2.0_simple/sh_v2_simple.xacro"/>
-  <xacro:macro name="softhands" params="type version parent position orientation operation_mode translation fixed_hands:='false'">
+  <xacro:macro name="softhands" params="type version parent position orientation operation_mode translation fixed_hands:='false' useCollisionMesh:='true' ">
     # Softhand VERSION 1.0
     <xacro:if value="${version == 'v1.0'}">
@@ -59,5 +59,6 @@
         orientation ="${orientation}"
         operation_mode = "${operation_mode}"
-        fixed_hand = "${fixed_hands}">
+        fixed_hand = "${fixed_hands}"
+        useCollisionMesh = "${useCollisionMesh}">
       </xacro:sh_v1_simple>
     </xacro:if>

File: softhands_description/urdf/v1.0_simple/finger.xacro (robot description, xacro)
@@ -38,5 +38,5 @@
 -->
 <robot xmlns:xacro="http://www.ros.org/wiki/xacro">
-  <xacro:macro name="finger_v1_simple" params="type ns sign position orientation fixed:='false'">
+  <xacro:macro name="finger_v1_simple" params="type ns sign position orientation fixed:='false' useCollisionMesh:='true' ">
   <xacro:if value="${fixed == False}">
     <xacro:property name="joint_type" value="revolute"/>
@@ -65,4 +65,5 @@
         </geometry>
       </visual>
+      <xacro:if value="${useCollisionMesh}">
       <collision>
         <geometry>
@@ -70,4 +71,5 @@
         </geometry>
       </collision>
+      </xacro:if>
     </link>
     <!-- PROXIMAL PHALANGE -->
@@ -90,4 +92,5 @@
         </geometry>
       </visual>
+      <xacro:if value="${useCollisionMesh}">
       <collision>
         <geometry>
@@ -95,4 +98,5 @@
         </geometry>
       </collision>
+      </xacro:if>
     </link>
     <!-- MIDDLE PHALANGE -->
@@ -116,4 +120,5 @@
         </geometry>
       </visual>
+      <xacro:if value="${useCollisionMesh}">
       <collision>
         <geometry>
@@ -121,4 +126,5 @@
         </geometry>
       </collision>
+      </xacro:if>
     </link>
     <!-- DISTAL PHALANGE -->
@@ -142,4 +148,5 @@
         </geometry>
       </visual>
+      <xacro:if value="${useCollisionMesh}">
       <collision>
         <geometry>
@@ -147,4 +154,5 @@
         </geometry>
       </collision>
+      </xacro:if>
     </link>
   </xacro:macro>

File: softhands_description/urdf/v1.0_simple/sh_v1_simple.xacro (robot description, xacro)
@@ -40,5 +40,5 @@
 	<xacro:include filename="$(find softhands_description)/urdf/v1.0_simple/finger.xacro" />
 	<xacro:include filename="$(find softhands_description)/urdf/v1.0_simple/thumb.xacro" />
-	<xacro:macro name="sh_v1_simple" params="type parent position orientation operation_mode fixed_hand:='false'">
+	<xacro:macro name="sh_v1_simple" params="type parent position orientation operation_mode fixed_hand:='false' useCollisionMesh:='true' ">
 		# Softhand Base
 		<joint name="${type}_hand_base_joint" type="fixed">
@@ -67,32 +67,34 @@
 					</geometry>
 				</visual>
-				<collision>
-					<geometry>
-						<mesh filename="package://softhands_description/meshes/softhands/v1.0/right/palm_right_m.stl" />
-					</geometry>
-				</collision>
-				<visual>
-					<origin xyz="-0.002 -0.00695 -0.0535" rpy="0 0 0" />
-					<geometry>
-						<mesh filename="package://softhands_description/meshes/softhands/v1.0/right/softhand_base_right_m.stl" />
-					</geometry>
-				</visual>
-				<collision>
-					<origin xyz="-0.002 -0.00695 -0.0535" rpy="0 0 0" />
-					<geometry>
-						<mesh filename="package://softhands_description/meshes/softhands/v1.0/right/softhand_base_right_m.stl" />
-					</geometry>
-				</collision>
+				<xacro:if value="${useCollisionMesh}">
+					<collision>
+						<geometry>
+							<mesh filename="package://softhands_description/meshes/softhands/v1.0/right/palm_right_m.stl" />
+						</geometry>
+					</collision>
+					<visual>
+						<origin xyz="-0.002 -0.00695 -0.0535" rpy="0 0 0" />
+						<geometry>
+							<mesh filename="package://softhands_description/meshes/softhands/v1.0/right/softhand_base_right_m.stl" />
+						</geometry>
+					</visual>
+					<collision>
+						<origin xyz="-0.002 -0.00695 -0.0535" rpy="0 0 0" />
+						<geometry>
+							<mesh filename="package://softhands_description/meshes/softhands/v1.0/right/softhand_base_right_m.stl" />
+						</geometry>
+					</collision>
+				</xacro:if>
 			</link>
 			# Thumb finger
-			<xacro:thumb_v1_simple type="thumb" ns="${type}_hand_v1s" sign="1" position="0.00566972 0.0296160 0.0553140" orientation="0.0 -0.38397275793662144 1.5707963267948966" fixed="${fixed_hand}"></xacro:thumb_v1_simple>
+			<xacro:thumb_v1_simple type="thumb" ns="${type}_hand_v1s" sign="1" position="0.00566972 0.0296160 0.0553140" orientation="0.0 -0.38397275793662144 1.5707963267948966" fixed="${fixed_hand}" useCollisionMesh="${useCollisionMesh}"></xacro:thumb_v1_simple>
 			# Index finger
-			<xacro:finger_v1_simple type="index" ns="${type}_hand_v1s" sign="1" position="-0.0033 0.0195 0.0936994" orientation="1.5707963267948966 -1.4835299330931884 1.5707963267948966" fixed="${fixed_hand}"></xacro:finger_v1_simple>
+			<xacro:finger_v1_simple type="index" ns="${type}_hand_v1s" sign="1" position="-0.0033 0.0195 0.0936994" orientation="1.5707963267948966 -1.4835299330931884 1.5707963267948966" fixed="${fixed_hand}" useCollisionMesh="${useCollisionMesh}"></xacro:finger_v1_simple>
 			# Middle finger
-			<xacro:finger_v1_simple type="middle" ns="${type}_hand_v1s" sign="1" position="-0.003300000 0.0 0.100699" orientation="3.141592 -1.5707963267948966 0.0" fixed="${fixed_hand}"></xacro:finger_v1_simple>
+			<xacro:finger_v1_simple type="middle" ns="${type}_hand_v1s" sign="1" position="-0.003300000 0.0 0.100699" orientation="3.141592 -1.5707963267948966 0.0" fixed="${fixed_hand}" useCollisionMesh="${useCollisionMesh}"></xacro:finger_v1_simple>
 			# Ring finger
-			<xacro:finger_v1_simple type="ring" ns="${type}_hand_v1s" sign="1" position="-0.0033 -0.0195 0.0936994" orientation="-1.5707963267948966 -1.5184364298870514 -1.5707963267948966" fixed="${fixed_hand}"></xacro:finger_v1_simple>
+			<xacro:finger_v1_simple type="ring" ns="${type}_hand_v1s" sign="1" position="-0.0033 -0.0195 0.0936994" orientation="-1.5707963267948966 -1.5184364298870514 -1.5707963267948966" fixed="${fixed_hand}" useCollisionMesh="${useCollisionMesh}"></xacro:finger_v1_simple>
 			# Little finger
-			<xacro:finger_v1_simple type="little" ns="${type}_hand_v1s" sign="1" position="-0.0033 -0.039 0.0836994" orientation="-1.5707963267948966 -1.4835299330931884 -1.5707963267948966" fixed="${fixed_hand}"></xacro:finger_v1_simple>
+			<xacro:finger_v1_simple type="little" ns="${type}_hand_v1s" sign="1" position="-0.0033 -0.039 0.0836994" orientation="-1.5707963267948966 -1.4835299330931884 -1.5707963267948966" fixed="${fixed_hand}" useCollisionMesh="${useCollisionMesh}"></xacro:finger_v1_simple>
 			<!-- grasp joint -->
 		<joint name="${type}_hand_v1s_grasp_joint" type="fixed">
@@ -123,32 +125,34 @@
 					</geometry>
 				</visual>
-				<collision>
-					<geometry>
-						<mesh filename="package://softhands_description/meshes/softhands/v1.0/left/palm_left_m.stl" />
-					</geometry>
-				</collision>
-				<visual>
-					<origin xyz="-0.002 0.00695 -0.0535" rpy="0 0 0" />
-					<geometry>
-						<mesh filename="package://softhands_description/meshes/softhands/v1.0/left/softhand_base_left_m.stl" />
-					</geometry>
-				</visual>
-				<collision>
-					<origin xyz="-0.002 0.00695 -0.0535" rpy="0 0 0" />
-					<geometry>
-						<mesh filename="package://softhands_description/meshes/softhands/v1.0/right/softhand_base_right_m.stl" />
-					</geometry>
-				</collision>
+				<xacro:if value="${useCollisionMesh}">
+					<collision>
+						<geometry>
+							<mesh filename="package://softhands_description/meshes/softhands/v1.0/left/palm_left_m.stl" />
+						</geometry>
+					</collision>
+					<visual>
+						<origin xyz="-0.002 0.00695 -0.0535" rpy="0 0 0" />
+						<geometry>
+							<mesh filename="package://softhands_description/meshes/softhands/v1.0/left/softhand_base_left_m.stl" />
+						</geometry>
+					</visual>
+					<collision>
+						<origin xyz="-0.002 0.00695 -0.0535" rpy="0 0 0" />
+						<geometry>
+							<mesh filename="package://softhands_description/meshes/softhands/v1.0/right/softhand_base_right_m.stl" />
+						</geometry>
+					</collision>
+				</xacro:if>
 			</link>
 			# Thumb finger
-			<xacro:thumb_v1_simple type="thumb" ns="${type}_hand_v1s" sign="-1" position="0.005669722 -0.029616 0.055314" orientation="0.0 -0.38397275793662144 -1.5707963267948966" fixed="${fixed_hand}"></xacro:thumb_v1_simple>
+			<xacro:thumb_v1_simple type="thumb" ns="${type}_hand_v1s" sign="-1" position="0.005669722 -0.029616 0.055314" orientation="0.0 -0.38397275793662144 -1.5707963267948966" fixed="${fixed_hand}" useCollisionMesh="${useCollisionMesh}"></xacro:thumb_v1_simple>
 			# Index finger
-			<xacro:finger_v1_simple type="index" ns="${type}_hand_v1s" sign="-1" position="-0.0033 -0.0195 0.0936994" orientation="-1.5707963267948966 -1.4835299330931884 -1.5707963267948966" fixed="${fixed_hand}"></xacro:finger_v1_simple>
+			<xacro:finger_v1_simple type="index" ns="${type}_hand_v1s" sign="-1" position="-0.0033 -0.0195 0.0936994" orientation="-1.5707963267948966 -1.4835299330931884 -1.5707963267948966" fixed="${fixed_hand}" useCollisionMesh="${useCollisionMesh}"></xacro:finger_v1_simple>
 			# Middle finger
-			<xacro:finger_v1_simple type="middle" ns="${type}_hand_v1s" sign="-1" position="-0.0033 0.0 0.100699" orientation="3.1415 -1.5707963267948966 0.0" fixed="${fixed_hand}"></xacro:finger_v1_simple>
+			<xacro:finger_v1_simple type="middle" ns="${type}_hand_v1s" sign="-1" position="-0.0033 0.0 0.100699" orientation="3.1415 -1.5707963267948966 0.0" fixed="${fixed_hand}" useCollisionMesh="${useCollisionMesh}"></xacro:finger_v1_simple>
 			# Ring finger
-			<xacro:finger_v1_simple type="ring" ns="${type}_hand_v1s" sign="-1" position="-0.0033 0.0195 0.0936994" orientation="1.5707963267948966 -1.5184364298870514 1.5707963267948966" fixed="${fixed_hand}"></xacro:finger_v1_simple>
+			<xacro:finger_v1_simple type="ring" ns="${type}_hand_v1s" sign="-1" position="-0.0033 0.0195 0.0936994" orientation="1.5707963267948966 -1.5184364298870514 1.5707963267948966" fixed="${fixed_hand}" useCollisionMesh="${useCollisionMesh}"></xacro:finger_v1_simple>
 			# Little finger
-			<xacro:finger_v1_simple type="little" ns="${type}_hand_v1s" sign="-1" position="-0.0033 0.039 0.0836994" orientation="1.5707963267948966 -1.4835299330931884 1.5707963267948966" fixed="${fixed_hand}"></xacro:finger_v1_simple>
+			<xacro:finger_v1_simple type="little" ns="${type}_hand_v1s" sign="-1" position="-0.0033 0.039 0.0836994" orientation="1.5707963267948966 -1.4835299330931884 1.5707963267948966" fixed="${fixed_hand}" useCollisionMesh="${useCollisionMesh}"></xacro:finger_v1_simple>
 		<!-- grasp joint -->
 		<joint name="${type}_hand_v1s_grasp_joint" type="fixed">

File: softhands_description/urdf/v1.0_simple/thumb.xacro (robot description, xacro)
@@ -38,5 +38,5 @@
 -->
 <robot xmlns:xacro="http://www.ros.org/wiki/xacro">
-  <xacro:macro name="thumb_v1_simple" params="type ns sign position orientation fixed:='false'">
+  <xacro:macro name="thumb_v1_simple" params="type ns sign position orientation fixed:='false' useCollisionMesh:='true' ">
   <xacro:if value="${fixed == False}">
     <xacro:property name="joint_type" value="continuous"/>
@@ -65,4 +65,5 @@
           </geometry>
         </visual>
+        <xacro:if value="${useCollisionMesh}">
         <collision>
           <geometry>
@@ -70,4 +71,5 @@
           </geometry>
         </collision>
+        </xacro:if>
       </xacro:if>
       <xacro:if value="${ns == 'left_hand_v1s'}">
@@ -77,4 +79,5 @@
           </geometry>
         </visual>
+        <xacro:if value="${useCollisionMesh}">
         <collision>
           <geometry>
@@ -82,4 +85,5 @@
           </geometry>
         </collision>
+        </xacro:if>
       </xacro:if>
     </link>
@@ -103,4 +107,5 @@
         </geometry>
       </visual>
+      <xacro:if value="${useCollisionMesh}">
       <collision>
         <geometry>
@@ -108,4 +113,5 @@
         </geometry>
       </collision>
+      </xacro:if>
     </link>
     <!-- DISTAL PHALANGE -->
@@ -128,4 +134,5 @@
         </geometry>
       </visual>
+      <xacro:if value="${useCollisionMesh}">
       <collision>
         <geometry>
@@ -133,4 +140,5 @@
         </geometry>
       </collision>
+      </xacro:if>
     </link>
   </xacro:macro>
