Commit message: added grasp point and mimic params for gazebo

File: softhands_description/urdf/v1.0_simple/sh_v1_simple.xacro (robot description, xacro)
@@ -144,4 +144,14 @@
 			<xacro:finger_v1_simple type="little" ns="${type}_hand_v1s" sign="-1" position="-0.0033 0.039 0.0836994" orientation="1.5707963267948966 -1.4835299330931884 1.5707963267948966" fixed="${fixed_hand}"></xacro:finger_v1_simple>
 		</xacro:if>
+		<!-- grasp joint -->
+		<joint name="${type}_hand_v1s_grasp_joint" type="fixed">
+			<origin xyz="0.0 0.0 0.07" rpy="0 0 0" />
+			<parent link="${type}_hand_v1s_palm_link" />
+			<child link="${type}_hand_v1s_grasp_link" />
+		</joint>
+		<link name="${type}_hand_v1s_grasp_link" />
+		<gazebo reference="${type}_hand_v1s_grasp_link">
+			<material>Gazebo/White</material>
+		</gazebo>
 		# Gazebo NEW custom synergy-plugin
 		<gazebo>
@@ -149,4 +159,57 @@
 				<namespace>${type}_hand_v1s</namespace>
 				<operation_mode>${operation_mode}</operation_mode>
+				<!-- Optional parameter to fit with the real EGO's arm -->
+				<r_finger>0.0033</r_finger>
+				<R_pulley>0.0053</R_pulley>
+				<n_param>0.058</n_param> <!-- The formula is (4*r_finger)/(2*R_pulley) -->
+				<spring_k>0.5</spring_k>
+				<!-- Parameters for synergy matrix (S) -->
+				<synS_thumb_j1>1.2</synS_thumb_j1>
+				<synS_thumb_j2>1.2</synS_thumb_j2>
+				<synS_thumb_j3>1.2</synS_thumb_j3>
+				<k_thumb_j1>0.8</k_thumb_j1>
+				<k_thumb_j2>0.8</k_thumb_j2>
+				<k_thumb_j3>0.8</k_thumb_j3>
+				<synS_index_j2>1.57</synS_index_j2>
+				<synS_index_j3>1.25</synS_index_j3>
+				<synS_index_j4>0.8</synS_index_j4>
+				<k_index_j1>0.25</k_index_j1>
+				<k_index_j2>0.5</k_index_j2>
+				<k_index_j3>0.5</k_index_j3>
+				<k_index_j4>0.5</k_index_j4>
+				<synS_middle_j2>1.57</synS_middle_j2>
+				<synS_middle_j3>1.25</synS_middle_j3>
+				<synS_middle_j4>1.25</synS_middle_j4>
+				<k_middle_j1>0.25</k_middle_j1>
+				<k_middle_j2>0.5</k_middle_j2>
+				<k_middle_j3>0.5</k_middle_j3>
+				<k_middle_j4>0.5</k_middle_j4>
+				<synS_ring_j2>1.57</synS_ring_j2>
+				<synS_ring_j3>1.0</synS_ring_j3>
+				<synS_ring_j4>1.0</synS_ring_j4>
+				<k_ring_j1>0.25</k_ring_j1>
+				<k_ring_j2>0.5</k_ring_j2>
+				<k_ring_j3>0.5</k_ring_j3>
+				<k_ring_j4>0.5</k_ring_j4>
+				<synS_little_j2>1.57</synS_little_j2>
+				<synS_little_j3>1.25</synS_little_j3>
+				<synS_little_j4>1.0</synS_little_j4>
+				<k_little_j1>0.25</k_little_j1>
+				<k_little_j2>0.5</k_little_j2>
+				<k_little_j3>0.5</k_little_j3>
+				<k_little_j4>0.5</k_little_j4>
+				<!-- Change tags sign according to the hand type -->
+				<xacro:if value="${type == 'right'}">
+					<synS_index_j1>0.3</synS_index_j1>
+					<synS_middle_j1>0</synS_middle_j1>
+					<synS_ring_j1>0</synS_ring_j1>
+					<synS_little_j1>-0.2</synS_little_j1>
+				</xacro:if>
+				<xacro:if value="${type == 'left'}">
+					<synS_index_j1>-0.3</synS_index_j1>
+					<synS_middle_j1>0</synS_middle_j1>
+					<synS_ring_j1>0</synS_ring_j1>
+					<synS_little_j1>0.1</synS_little_j1>
+				</xacro:if>
 			</plugin>
 		</gazebo>

Commit message: changed grasping point

File: softhands_description/urdf/v1.0_simple/sh_v1_simple.xacro (robot description, xacro)
@@ -95,4 +95,12 @@
 			# Little finger
 			<xacro:finger_v1_simple type="little" ns="${type}_hand_v1s" sign="1" position="-0.0033 -0.039 0.0836994" orientation="-1.5707963267948966 -1.4835299330931884 -1.5707963267948966" fixed="${fixed_hand}"></xacro:finger_v1_simple>
+			<!-- grasp joint -->
+		<joint name="${type}_hand_v1s_grasp_joint" type="fixed">
+			<origin xyz="0.03 0.06 0.10" rpy="0 0 0" />
+			<parent link="${type}_hand_v1s_palm_link" />
+			<child link="${type}_hand_v1s_grasp_link" />
+		</joint>
+		<link name="${type}_hand_v1s_grasp_link">
+		</link>
 		</xacro:if>
 		# LEFT HAND
@@ -143,4 +151,15 @@
 			# Little finger
 			<xacro:finger_v1_simple type="little" ns="${type}_hand_v1s" sign="-1" position="-0.0033 0.039 0.0836994" orientation="1.5707963267948966 -1.4835299330931884 1.5707963267948966" fixed="${fixed_hand}"></xacro:finger_v1_simple>
+		<!-- grasp joint -->
+		<joint name="${type}_hand_v1s_grasp_joint" type="fixed">
+			<origin xyz="0.03 -0.06 0.10" rpy="0 0 0" />
+			<parent link="${type}_hand_v1s_palm_link" />
+			<child link="${type}_hand_v1s_grasp_link" />
+		</joint>
+		<link name="${type}_hand_v1s_grasp_link">
+		</link>
+		<gazebo reference="${type}_hand_v1s_grasp_link">
+			<material>Gazebo/White</material>
+		</gazebo>
 		</xacro:if>
 		# Gazebo NEW custom synergy-plugin

Commit message: bug fix

File: softhands_description/urdf/v1.0_simple/sh_v1_simple.xacro (robot description, xacro)
@@ -73,5 +73,6 @@
 						</geometry>
 					</collision>
-					<visual>
+				</xacro:if>
+				<visual>
 						<origin xyz="-0.002 -0.00695 -0.0535" rpy="0 0 0" />
 						<geometry>
@@ -79,4 +80,5 @@
 						</geometry>
 					</visual>
+				<xacro:if value="${useCollisionMesh}">
 					<collision>
 						<origin xyz="-0.002 -0.00695 -0.0535" rpy="0 0 0" />
@@ -131,5 +133,6 @@
 						</geometry>
 					</collision>
-					<visual>
+				</xacro:if>
+				<visual>
 						<origin xyz="-0.002 0.00695 -0.0535" rpy="0 0 0" />
 						<geometry>
@@ -137,4 +140,5 @@
 						</geometry>
 					</visual>
+				<xacro:if value="${useCollisionMesh}">
 					<collision>
 						<origin xyz="-0.002 0.00695 -0.0535" rpy="0 0 0" />
